Commit message: added image_process node

File: catkin_ws/src/my_robot/urdf/my_robot.xacro (robot description, xacro)
@@ -64,5 +64,5 @@
 	  </visual>
     <collision name = 'right_wheel_collision'>
-		  <origin xyz="0 0 0" rpy = "0 1.5707 1.5707"/>
+		  <origin xyz="0 0.15 0" rpy = "0 1.5707 1.5707"/>
       <geometry>
         <cylinder radius = '0.1' length = '0.05'/>
@@ -79,5 +79,5 @@
     </inertial>
   </link>
-  <joint name = "right_wheel_joint" type = "continuous">
+  <joint name = "right_wheel_hinge" type = "continuous">
     <origin xyz = "0 0 0" rpy = "0 0 0" />
     <child link = "right_wheel"/>
@@ -95,5 +95,5 @@
 	  </visual>
     <collision name = 'left_wheel_collision'>
-		  <origin xyz="0 0 0" rpy = "0 1.5707 1.5707"/>
+		  <origin xyz="0 -0.15 0" rpy = "0 1.5707 1.5707"/>
       <geometry>
         <cylinder radius = '0.1' length = '0.05'/>
@@ -110,5 +110,5 @@
     </inertial>
   </link>
-  <joint name = "left_wheel_joint" type = "continuous">
+  <joint name = "left_wheel_hinge" type = "continuous">
     <origin xyz = "0 0 0" rpy = "0 0 0" />
     <child link = "left_wheel"/>
@@ -120,5 +120,5 @@
   <link name = 'camera'>
 	  <visual name = 'camera_visual'>
-		  <origin xyz="0.2 0 0" rpy = "0 0 0"/>
+		  <origin xyz="0 0 0" rpy = "0 0 0"/>
       <geometry>
         <box size = "0.05 0.05 0.05"/>
@@ -126,5 +126,5 @@
 	  </visual>
     <collision name = 'camera_collision'>
-		  <origin xyz="0.2 0 0" rpy = "0 0 0"/>
+		  <origin xyz="0 0 0" rpy = "0 0 0"/>
       <geometry>
         <box size = "0.05 0.05 0.05"/>
@@ -133,5 +133,4 @@
     <inertial name = 'camera_inertial'>
       <mass value="0.1"/>
-      <origin xyz="0.05 0.05 0.05" rpy = "0 0 0"/>
       <inertia
           ixx="1e-6" ixy="0" ixz="0"
@@ -142,10 +141,10 @@
   </link>
   <joint name = "camera_joint" type = "fixed">
-    <origin xyz = "0 0 0" rpy = "0 0 0" />
+    <origin xyz = "0.2 0 0" rpy = "0 0 0" />
     <child link = "camera"/>
     <parent link = "chassis"/>
     <axis xyz = "0 1 0" rpy = "0 0 0"/>
   </joint>
-<link name = 'hokuyo'>
+  <link name = 'hokuyo'>
 	  <visual name = 'hokuyo_visual'>
 		  <origin xyz="0.15 0 0.1" rpy = "0 0 0"/>

Commit message: Made some changes to image_process node but it still doesn't work

File: catkin_ws/src/my_robot/urdf/my_robot.xacro (robot description, xacro)
@@ -174,3 +174,13 @@
     <axis xyz = "0 1 0" rpy = "0 0 0"/>
   </joint>
+<!-- coloring the robot> <!-->
+  <gazebo reference = "chassis">
+    <material>Gazebo/Yellow</material>
+  </gazebo>
+  <gazebo reference = "left_wheel">
+    <material>Gazebo/Black</material>
+  </gazebo>
+  <gazebo reference = "right_wheel">
+    <material>Gazebo/Black</material>
+  </gazebo>
 </robot>
